Commit message: 

File: trunk/car_like_simulation/car_like.urdf.xacro (robot description, xacro)
@@ -25,12 +25,12 @@
     <link name="base_link">
         <inertial>
-            <mass value="1.0" />
-            <origin xyz="0 0 0" />
-            <inertia  ixx="1.0" ixy="0.0"  ixz="0.0"  iyy="1.0"  iyz="0.0"  izz="1.0" />
+            <mass value="0.2" />
+            <origin xyz="0 0 0" />
+            <inertia  ixx="0.2" ixy="0.0"  ixz="0.0"  iyy="0.2"  iyz="0.0"  izz="0.2" />
         </inertial>
         <visual>
             <origin xyz="0 0 0" rpy="0 0 0" />
             <geometry>
-                <box size="2.0 1.0 0.1" />
+                <box size="0.4 0.15 0.1" />
             </geometry>
             <material name="Blue"/>
@@ -39,5 +39,5 @@
             <origin xyz="0 0 0" rpy="0 0 0" />
             <geometry>
-                <box size="2.0 1.0 0.1" />
+                <box size="0.4 0.15 0.1" />
             </geometry>
         </collision>
@@ -50,15 +50,15 @@
     	<parent link="base_link"/>
     	<child link="front_link"/>
-    	<origin xyz="0.8 0.0 -0.25"/>
+    	<origin xyz="0.16 0.0 -0.1"/>
     </joint>
     <link name="front_link">
         <inertial>
-            <mass value="1.0" />
-            <origin xyz="0 0 0" />
-            <inertia  ixx="1.0" ixy="0.0"  ixz="0.0"  iyy="1.0"  iyz="0.0"  izz="1.0" />
-        </inertial>
-        <visual>
-            <geometry>
-                <box size="0.1 1.0 0.01" />
+            <mass value="0.01" />
+            <origin xyz="0 0 0" />
+            <inertia  ixx="0.01" ixy="0.0"  ixz="0.0"  iyy="0.01"  iyz="0.0"  izz="0.01" />
+        </inertial>
+        <visual>
+            <geometry>
+                <box size="0.02 0.15 0.005" />
             </geometry>
             <material name="Red"/>
@@ -66,5 +66,5 @@
         <collision>
             <geometry>
-                <box size="0.1 1.0 0.01" />
+                <box size="0.02 0.15 0.005" />
             </geometry>
         </collision>
@@ -83,19 +83,19 @@
     <link name="steer_link">
         <inertial>
-            <mass value="1.0" />
-            <origin xyz="0 0 0" />
-            <inertia  ixx="1.0" ixy="0.0"  ixz="0.0"  iyy="1.0"  iyz="0.0"  izz="1.0" />
-        </inertial>
-        <visual>
-            <origin xyz="-0.15 0 0" />
-            <geometry>
-                <box size="0.4 0.1 0.01" />
+            <mass value="0.01" />
+            <origin xyz="0 0 0" />
+            <inertia  ixx="0.01" ixy="0.0"  ixz="0.0"  iyy="0.01"  iyz="0.0"  izz="0.01" />
+        </inertial>
+        <visual>
+            <origin xyz="-0.02 0 0" />
+            <geometry>
+                <box size="0.04 0.02 0.005" />
             </geometry>
             <material name="Red"/>
         </visual>
         <collision>
-            <origin xyz="-0.15 0 0" />
-            <geometry>
-                <box size="0.4 0.1 0.01" />
+            <origin xyz="0.02 0 0" />
+            <geometry>
+                <box size="0.04 0.02 0.005" />
             </geometry>
         </collision>
@@ -110,23 +110,23 @@
         <parent link="front_link" />
         <child link="front_left_bar_link" />
-        <origin xyz="0.0 0.45 0.0" rpy="0 0 0" />
+        <origin xyz="0.0 0.06 0.0" rpy="0 0 0" />
     </joint>
     <link name="front_left_bar_link">
         <inertial>
-            <mass value="1.0" />
-            <origin xyz="0 0 0" />
-            <inertia  ixx="1.0" ixy="0.0"  ixz="0.0"  iyy="1.0"  iyz="0.0"  izz="1.0" />
-        </inertial>
-        <visual>
-            <origin xyz="-0.15 0 0" />
-            <geometry>
-                <box size="0.4 0.1 0.01" />
+            <mass value="0.01" />
+            <origin xyz="0 0 0" />
+            <inertia  ixx="0.01" ixy="0.0"  ixz="0.0"  iyy="0.01"  iyz="0.0"  izz="0.01" />
+        </inertial>
+        <visual>
+            <origin xyz="-0.02 0 0" />
+            <geometry>
+                <box size="0.04 0.02 0.005" />
             </geometry>
             <material name="Red"/>
         </visual>
         <collision>
-            <origin xyz="-0.15 0 0" />
-            <geometry>
-                <box size="0.4 0.1 0.01" />
+            <origin xyz="-0.02 0 0" />
+            <geometry>
+                <box size="0.04 0.02 0.005" />
             </geometry>
         </collision>
@@ -141,23 +141,23 @@
         <parent link="front_link" />
         <child link="front_right_bar_link" />
-        <origin xyz="0.0 -0.45 0.0" rpy="0 0 0" />
+        <origin xyz="0.0 -0.06 0.0" rpy="0 0 0" />
     </joint>
     <link name="front_right_bar_link">
         <inertial>
-            <mass value="1.0" />
-            <origin xyz="0 0 0" />
-            <inertia  ixx="1.0" ixy="0.0"  ixz="0.0"  iyy="1.0"  iyz="0.0"  izz="1.0" />
-        </inertial>
-        <visual>
-            <origin xyz="-0.15 0 0" />
-            <geometry>
-                <box size="0.4 0.1 0.01" />
+            <mass value="0.01" />
+            <origin xyz="0 0 0" />
+            <inertia  ixx="0.01" ixy="0.0"  ixz="0.0"  iyy="0.01"  iyz="0.0"  izz="0.01" />
+        </inertial>
+        <visual>
+            <origin xyz="-0.02 0 0" />
+            <geometry>
+                <box size="0.04 0.02 0.005" />
             </geometry>
             <material name="Red"/>
         </visual>
         <collision>
-            <origin xyz="-0.15 0 0" />
-            <geometry>
-                <box size="0.4 0.1 0.01" />
+            <origin xyz="-0.02 0 0" />
+            <geometry>
+                <box size="0.04 0.02 0.005" />
             </geometry>
         </collision>
@@ -171,16 +171,16 @@
         <parent link="front_left_bar_link" />
         <child link="front_left_wheel_link" />
-        <origin xyz="0 0.1 0" rpy="0 0 0" />
+        <origin xyz="0 0.04 0" rpy="0 0 0" />
     </joint>
     <link name="front_left_wheel_link">
         <inertial>
-            <mass value="1.0" />
-            <origin xyz="0 0 0" />
-            <inertia  ixx="1.0" ixy="0.0"  ixz="0.0"  iyy="1.0"  iyz="0.0"  izz="1.0" />
-        </inertial>
-        <visual>
-            <origin xyz="0 0 0" rpy="${M_PI/2} 0 0" />
-            <geometry>
-                <cylinder radius="0.2" length="0.01" />
+            <mass value="0.01" />
+            <origin xyz="0 0 0" />
+            <inertia  ixx="0.01" ixy="0.0"  ixz="0.0"  iyy="0.01"  iyz="0.0"  izz="0.01" />
+        </inertial>
+        <visual>
+            <origin xyz="0 0 0" rpy="${M_PI/2} 0 0" />
+            <geometry>
+                <cylinder radius="0.02" length="0.005" />
             </geometry>
             <material name="Green"/>
@@ -189,5 +189,5 @@
             <origin xyz="0 0 0" rpy="${M_PI/2} 0 0" />
             <geometry>
-                <cylinder radius="0.2" length="0.01" />
+                <cylinder radius="0.02" length="0.005" />
             </geometry>
         </collision>
@@ -201,16 +201,16 @@
         <parent link="front_right_bar_link" />
         <child link="front_right_wheel_link" />
-        <origin xyz="0 -0.1 0" rpy="0 0 0" />
+        <origin xyz="0 -0.04 0" rpy="0 0 0" />
     </joint>
     <link name="front_right_wheel_link">
         <inertial>
-            <mass value="1.0" />
-            <origin xyz="0 0 0" />
-            <inertia  ixx="1.0" ixy="0.0"  ixz="0.0"  iyy="1.0"  iyz="0.0"  izz="1.0" />
-        </inertial>
-        <visual>
-            <origin xyz="0 0 0" rpy="${M_PI/2} 0 0" />
-            <geometry>
-                <cylinder radius="0.2" length="0.01" />
+            <mass value="0.01" />
+            <origin xyz="0 0 0" />
+            <inertia  ixx="0.01" ixy="0.0"  ixz="0.0"  iyy="0.01"  iyz="0.0"  izz="0.01" />
+        </inertial>
+        <visual>
+            <origin xyz="0 0 0" rpy="${M_PI/2} 0 0" />
+            <geometry>
+                <cylinder radius="0.02" length="0.005" />
             </geometry>
             <material name="Green"/>
@@ -219,5 +219,5 @@
             <origin xyz="0 0 0" rpy="${M_PI/2} 0 0" />
             <geometry>
-                <cylinder radius="0.2" length="0.01" />
+                <cylinder radius="0.02" length="0.005" />
             </geometry>
         </collision>
@@ -233,15 +233,15 @@
         <parent link="steer_link" />
         <child link="ackermann_bar_link" />
-        <origin xyz="-0.3 0 0" rpy="0 0 0" />
+        <origin xyz="-0.04 0 0" rpy="0 0 0" />
     </joint>
     <link name="ackermann_bar_link">
         <inertial>
-            <mass value="1.0" />
-            <origin xyz="0 0 0" />
-            <inertia  ixx="1.0" ixy="0.0"  ixz="0.0"  iyy="1.0"  iyz="0.0"  izz="1.0" />
-        </inertial>
-        <visual>
-            <geometry>
-                <box size="0.1 1.0 0.01" />
+            <mass value="0.01" />
+            <origin xyz="0 0 0" />
+            <inertia  ixx="0.01" ixy="0.0"  ixz="0.0"  iyy="0.01"  iyz="0.0"  izz="0.01" />
+        </inertial>
+        <visual>
+            <geometry>
+                <box size="0.02 0.15 0.01" />
             </geometry>
             <material name="Red"/>
@@ -249,5 +249,5 @@
         <collision>
             <geometry>
-                <box size="0.1 1.0 0.01" />
+                <box size="0.02 0.15 0.01" />
             </geometry>
         </collision>
@@ -257,5 +257,5 @@
     </gazebo>
     <gazebo reference="ackermann_bar_link">
-        <material>Gazebo/Red</material>
+        <material>Gazebo/Blue</material>
     </gazebo>
 	<!-- Gazebo Ackermann loop joints -->
@@ -266,5 +266,5 @@
         <anchor>ackermann_bar_link</anchor>
         <axis>0 0 1</axis>
-        <anchorOffset>0 0.45 0</anchorOffset>
+        <anchorOffset>0 0.06 0</anchorOffset>
       </joint:hinge>
     </gazebo>
@@ -275,5 +275,5 @@
         <anchor>ackermann_bar_link</anchor>
         <axis>0 0 1</axis>
-        <anchorOffset>0 -0.45 0</anchorOffset>
+        <anchorOffset>0 -0.06 0</anchorOffset>
       </joint:hinge>
     </gazebo>
@@ -283,16 +283,16 @@
         <parent link="base_link" />
         <child link="back_left_wheel_link" />
-        <origin xyz="-0.8 0.55 -0.25" rpy="0 0 0" />
+        <origin xyz="-0.16 0.1 -0.1" rpy="0 0 0" />
     </joint>
     <link name="back_left_wheel_link">
         <inertial>
-            <mass value="1.0" />
-            <origin xyz="0 0 0" />
-            <inertia  ixx="1.0" ixy="0.0"  ixz="0.0"  iyy="1.0"  iyz="0.0"  izz="1.0" />
-        </inertial>
-        <visual>
-            <origin xyz="0 0 0" rpy="${M_PI/2} 0 0" />
-            <geometry>
-                <cylinder radius="0.2" length="0.01" />
+            <mass value="0.01" />
+            <origin xyz="0 0 0" />
+            <inertia  ixx="0.01" ixy="0.0"  ixz="0.0"  iyy="0.01"  iyz="0.0"  izz="0.01" />
+        </inertial>
+        <visual>
+            <origin xyz="0 0 0" rpy="${M_PI/2} 0 0" />
+            <geometry>
+                <cylinder radius="0.02" length="0.005" />
             </geometry>
             <material name="Green"/>
@@ -301,5 +301,5 @@
             <origin xyz="0 0 0" rpy="${M_PI/2} 0 0" />
             <geometry>
-                <cylinder radius="0.2" length="0.01" />
+                <cylinder radius="0.02" length="0.005" />
             </geometry>
         </collision>
@@ -313,16 +313,16 @@
         <parent link="base_link" />
         <child link="back_right_wheel_link" />
-        <origin xyz="-0.8 -0.55 -0.25" rpy="0 0 0" />
+        <origin xyz="-0.16 -0.1 -0.1" rpy="0 0 0" />
     </joint>
     <link name="back_right_wheel_link">
         <inertial>
-            <mass value="1.0" />
-            <origin xyz="0 0 0" />
-            <inertia  ixx="1.0" ixy="0.0"  ixz="0.0"  iyy="1.0"  iyz="0.0"  izz="1.0" />
-        </inertial>
-        <visual>
-            <origin xyz="0 0 0" rpy="${M_PI/2} 0 0" />
-            <geometry>
-                <cylinder radius="0.2" length="0.01" />
+            <mass value="0.01" />
+            <origin xyz="0 0 0" />
+            <inertia  ixx="0.01" ixy="0.0"  ixz="0.0"  iyy="0.01"  iyz="0.0"  izz="0.01" />
+        </inertial>
+        <visual>
+            <origin xyz="0 0 0" rpy="${M_PI/2} 0 0" />
+            <geometry>
+                <cylinder radius="0.02" length="0.005" />
             </geometry>
             <material name="Green"/>
@@ -331,5 +331,5 @@
             <origin xyz="0 0 0" rpy="${M_PI/2} 0 0" />
             <geometry>
-                <cylinder radius="0.2" length="0.01" />
+                <cylinder radius="0.02" length="0.005" />
             </geometry>
         </collision>
@@ -348,10 +348,10 @@
 	<rightJoint>back_right_wheel_joint</rightJoint>
 	<steerJoint>steer_joint</steerJoint>
-	<wheelSeparationWidth>2.12</wheelSeparationWidth>
-	<wheelSeparationLength>2.33918</wheelSeparationLength>
+	<wheelSeparationWidth>0.16</wheelSeparationWidth>
+	<wheelSeparationLength>0.32</wheelSeparationLength>
         <!-- Shouldn't this wheel diameter include the tire?
              (40 cm is about right for the bare rim)
           -->
-	<wheelDiameter>0.4</wheelDiameter>
+	<wheelDiameter>0.041</wheelDiameter>
 	<driveTorque>5</driveTorque>
 	<steerTorque>5</steerTorque>

Commit message: 

File: trunk/car_like_simulation/car_like.urdf.xacro (robot description, xacro)
@@ -25,7 +25,7 @@
     <link name="base_link">
         <inertial>
-            <mass value="0.2" />
-            <origin xyz="0 0 0" />
-            <inertia  ixx="0.2" ixy="0.0"  ixz="0.0"  iyy="0.2"  iyz="0.0"  izz="0.2" />
+            <mass value="0.4" />
+            <origin xyz="0 0 0" />
+            <inertia  ixx="0.4" ixy="0.0"  ixz="0.0"  iyy="0.4"  iyz="0.0"  izz="0.4" />
         </inertial>
         <visual>
@@ -349,5 +349,5 @@
 	<steerJoint>steer_joint</steerJoint>
 	<wheelSeparationWidth>0.16</wheelSeparationWidth>
-	<wheelSeparationLength>0.32</wheelSeparationLength>
+	<wheelSeparationLength>0.45</wheelSeparationLength>
         <!-- Shouldn't this wheel diameter include the tire?
              (40 cm is about right for the bare rim)
